File: E-Fidget.kicad_sch (KiCad schematic)
At the start: 91 parts, among them J1 Conn_01x02, J2 USB_B_Micro, J3 Barrel_Jack_MountingPin, M1 Motor_DC, M2 Motor_DC, M3 Motor_DC, M4 Motor_DC, M5 Motor_DC, M6 Motor_DC, M7 Motor_DC, M8 Motor_DC, Q1 BSS138, Q2 BSS138, Q3 BSS138, Q4 BSS138, Q5 BSS138, Q6 BSS138, Q7 BSS138, Q8 BSS138, U1 W25Q128JVS, U2 AP3211KTR-G1, U3 RP2040, U4 AS78L05RTR-G1, X1 ENCODER_ANO, Y1 12MHz

Commit message: Update to 2.0
Parts:
- removed C19: 0.1u, Capacitor_SMD:C_0805_2012Metric_Pad1.18x1.45mm_HandSolder, symbol Device:C_Small
- removed C22: 0.33u, Capacitor_SMD:C_0805_2012Metric_Pad1.18x1.45mm_HandSolder, symbol Device:C_Small
- removed C3: 10u, Capacitor_SMD:C_0805_2012Metric_Pad1.18x1.45mm_HandSolder, symbol Device:C
- removed C6: 22u, Capacitor_SMD:C_0805_2012Metric_Pad1.18x1.45mm_HandSolder, symbol Device:C
- removed D1: D_Small, E-Fidget:SC-59_Handsoldering_No_Pin3, symbol Device:D_Small
- removed J2: USB_B_Micro, E-Fidget:USB_Micro-B_Amphenol_10103594-0001LF_Horizontal_modified, symbol E-Fidget-rescue:USB_B_Micro-Connector
- removed J3: Barrel_Jack_MountingPin, E-Fidget:CUI_PJ-102AH, symbol Connector:PJ-102AH
- removed L1: 4.7u, E-Fidget:NR6028T4R7M, symbol Device:L
- removed TP1, TP10, TP2, TP3, TP4, TP5, TP6, TP7, TP8, TP9: TestPoint, TestPoint:TestPoint_Pad_D2.0mm, symbol Connector:TestPoint
- removed U2: AP3211KTR-G1, Package_TO_SOT_SMD:SOT-23-6_Handsoldering, symbol Regulator_Switching:AP3211KTR-G1
- removed U4: AS78L05RTR-G1, E-Fidget:AS78L05RTR-G1, symbol AS78L05RTR:AS78L05RTR-G1
- removed X1: ENCODER_ANO, E-Fidget:ENCODER_ANO, symbol encoder_ano:ENCODER_ANO
- added BT1: WAFER-PH2.0-2PWB, Connector_JST:JST_PH_S2B-PH-SM4-TB_1x02-1MP_P2.00mm_Horizontal, symbol Device:Battery
- added C3, C6: 10u, Capacitor_SMD:C_0805_2012Metric, symbol Device:C_Small
- added D1: IN-S63AT5A, LED_SMD:LED_0603_1608Metric, symbol Device:LED_Small
- added J2: DX07S016JA1R1500, Connector_USB:USB_C_Receptacle_JAE_DX07S016JA1R1500, symbol Connector:USB_C_Receptacle_USB2.0
- added J3: DNP, Connector_PinHeader_2.54mm:PinHeader_1x09_P2.54mm_Vertical, symbol Connector:Conn_01x09_Female
- added J4: DNP, Connector_PinHeader_2.54mm:PinHeader_2x03_P2.54mm_Vertical, symbol Connector:Conn_01x06_Female
- added R16, R17: 5.1k, Resistor_SMD:R_0805_2012Metric, symbol Device:R_Small_US
- added SW1, SW2, SW3: K2-1102DP-E4SW-04, Button_Switch_THT:SW_PUSH_6mm, symbol Switch:SW_Push
- added U2: TPAP2112K-3.3TRG1, Package_TO_SOT_SMD:SOT-23-5, symbol Regulator_Linear:AP2112K-3.3
- added U4: MCP73831T-2ACI/OT, Package_TO_SOT_SMD:SOT-23-5, symbol Battery_Management:MCP73831-2-OT
- C5: value 10n -> 10u; footprint Capacitor_SMD:C_0805_2012Metric_Pad1.18x1.45mm_HandSolder -> Capacitor_SMD:C_0805_2012Metric
- D10, D11, D12: value SK6812 -> DNP
- D2, D3, D4, D5, D6, D7, D8, D9: value D_Small -> BAT54-7-F
- F1: value 0ZCJ0075AF2E -> 0ZCJ0020FF2E; footprint Fuse:Fuse_1206_3216Metric_Pad1.42x1.75mm_HandSolder -> Fuse:Fuse_1206_3216Metric
- H1, H2, H3, H4: value MountingHole -> DNP
- M1, M2, M3, M4, M5, M6, M7, M8: value Motor_DC -> DNP; footprint Connector_Wire:SolderWire-0.1sqmm_1x02_P3.6mm_D0.4mm_OD1mm_Relief -> Connector_Wire:SolderWire-0.1sqmm_1x02_P3.6mm_D0.4mm_OD1mm
- Q1, Q2, Q3, Q4, Q5, Q6, Q7, Q8: value BSS138 -> DMG2302UK-7; footprint Package_TO_SOT_SMD:SOT-323_SC-70_Handsoldering -> Package_TO_SOT_SMD:SC-59
- R2: value DNF -> DNP
- R4: value 16.3k -> 5.1k; footprint Resistor_SMD:R_0805_2012Metric_Pad1.20x1.40mm_HandSolder -> Resistor_SMD:R_0805_2012Metric
- R5: value 49.9k -> 5.1k; footprint Resistor_SMD:R_0805_2012Metric_Pad1.20x1.40mm_HandSolder -> Resistor_SMD:R_0805_2012Metric
- U1: value W25Q128JVS -> W25Q16JVSSIQ
- Y1: value 12MHz -> 445C25D12M00000
Connections:
- net +9V is gone; now on an unnamed net: F1.1
- net +1V1: now also J4.3 (Pin_3)
- net +3V3: now also F1.2, J3.4 (Pin_4); no longer D2.1 (K), D3.1 (K), D4.1 (K), D5.1 (K), D6.1 (K), D7.1 (K), D8.1 (K), D9.1 (K), M1.1 (+), M2.1 (+), M3.1 (+), M4.1 (+), M5.1 (+), M6.1 (+), M7.1 (+), M8.1 (+), R5.2
- net +5V: now also J2.A4 (VBUS), J2.A9 (VBUS), J2.B4 (VBUS), J2.B9 (VBUS), J3.1 (Pin_1), U4.4 (VDD)
- net GND: now also C5.2, R4.2, R5.2, BT1.2 (-), C3.2, C6.2, J2.A1 (GND), J2.A12 (GND), J2.B1 (GND), J2.B12 (GND), J2.S1 (SHIELD), J4.6 (Pin_6), R16.2, R17.2, SW1.2, SW2.2, SW3.2, U2.2 (GND), U4.2 (VSS); no longer R4.1
- net GPIO0: now also J3.7 (Pin_7)
- net GPIO1: now also J3.8 (Pin_8)
- net GPIO2: now also J4.4 (Pin_4)
- net GPIO26_ADC0: now also J3.9 (Pin_9)
- net GPIO3: now also SW1.1
- net GPIO4: now also SW3.1
- net GPIO5: now also SW2.1
- net SWCLK: now also J3.5 (Pin_5)
- net SWD: now also J4.2 (Pin_2)
- net USB_D+: now also J2.A6 (D+), J2.B6 (D+), J3.2 (Pin_2)
- net USB_D-: now also J2.A7 (D-), J2.B7 (D-), J3.3 (Pin_3)
- net ~{USB_BOOT}: now also J4.5 (Pin_5)
- net at C5.1: now also U2.5 (VOUT)
- net at R5.1: now also J2.B5 (CC2); no longer R4.2
- net PIXEL_OUT: now reaches D12.2-DOUT (DO)
- net PIXEL_OUT: now also J4.1 (Pin_1)
- new net: D1.1 (K), R17.1
- new net: R16.1, U4.5 (PROG)
- new net: J2.A5 (CC1), R4.1
- new net: D1.2 (A), U4.1 (STAT)
- new net +BATT: BT1.1 (+), C3.1, C6.1, D2.1 (K), D3.1 (K), D4.1 (K), D5.1 (K), D6.1 (K), D7.1 (K), D8.1 (K), D9.1 (K), J3.6 (Pin_6), M1.1 (+), M2.1 (+), M3.1 (+), M4.1 (+), M5.1 (+), M6.1 (+), M7.1 (+), M8.1 (+), U2.1 (VIN), U4.3 (VBAT)
- no-connect marks 2 -> 3
Other:
- note removed: "Power"
- moved on the sheet: D5, M4, Q4, R11
